File: micarrizo-pad.sch (KiCad schematic (older format))
At the start: 5 parts

Commit message: create big switch
Parts:
- removed MX? (x5): MX-LED, symbol MX_Alps_Hybrid:MX-LED
- added D? (x8): D_Small, symbol Device:D_Small
- added MX? (x8): MX-NoLED, symbol MX_Alps_Hybrid:MX-NoLED
- added U?: The-Big-Switch, symbol MX_Alps_Hybrid:The-Big-Switch
Connections:
- wire segments 0 -> 8
Changed lines of the file:
@@
 EESchema Schematic File Version 4
+LIBS:micarrizo-pad-cache
 EELAYER 30 0
 EELAYER END
@@
 $EndDescr
 $Comp
-L MX_Alps_Hybrid:MX-LED MX?
-U 1 1 65D06555
-P 4600 3400
-F 0 "MX?" H 4682 3624 60  0000 C CNN
-F 1 "MX-LED" H 4682 3550 20  0000 C CNN
-F 2 "" H 3975 3375 60  0001 C CNN
-F 3 "" H 3975 3375 60  0001 C CNN
-	1    4600 3400
-	1    0    0    -1
-$EndComp
-$Comp
-L MX_Alps_Hybrid:MX-LED MX?
-U 1 1 65D07A7B
-P 5000 3400
-F 0 "MX?" H 5082 3624 60  0000 C CNN
-F 1 "MX-LED" H 5082 3550 20  0000 C CNN
-F 2 "" H 4375 3375 60  0001 C CNN
-F 3 "" H 4375 3375 60  0001 C CNN
-	1    5000 3400
-	1    0    0    -1
-$EndComp
-$Comp
-L MX_Alps_Hybrid:MX-LED MX?
-U 1 1 65D091CD
-P 5400 3850
-F 0 "MX?" H 5482 4074 60  0000 C CNN
-F 1 "MX-LED" H 5482 4000 20  0000 C CNN
-F 2 "" H 4775 3825 60  0001 C CNN
-F 3 "" H 4775 3825 60  0001 C CNN
-	1    5400 3850
-	1    0    0    -1
-$EndComp
-$Comp
-L MX_Alps_Hybrid:MX-LED MX?
-U 1 1 65D0AB11
-P 4600 3850
-F 0 "MX?" H 4682 4074 60  0000 C CNN
-F 1 "MX-LED" H 4682 4000 20  0000 C CNN
-F 2 "" H 3975 3825 60  0001 C CNN
-F 3 "" H 3975 3825 60  0001 C CNN
-	1    4600 3850
-	1    0    0    -1
-$EndComp
-$Comp
-L MX_Alps_Hybrid:MX-LED MX?
-U 1 1 65D0B896
-P 5000 3850
-F 0 "MX?" H 5082 4074 60  0000 C CNN
-F 1 "MX-LED" H 5082 4000 20  0000 C CNN
-F 2 "" H 4375 3825 60  0001 C CNN
-F 3 "" H 4375 3825 60  0001 C CNN
-	1    5000 3850
-	1    0    0    -1
-$EndComp
+L MX_Alps_Hybrid:MX-NoLED MX?
+U 1 1 65EE9E93
+P 4250 3900
+F 0 "MX?" H 4283 4123 60  0000 C CNN
+F 1 "MX-NoLED" H 4283 4049 20  0000 C CNN
+F 2 "" H 3625 3875 60  0001 C CNN
+F 3 "" H 3625 3875 60  0001 C CNN
+	1    4250 3900
+	1    0    0    -1
+$EndComp
+$Comp
+L Device:D_Small D?
+U 1 1 65EEA4A1
+P 4100 4150
+F 0 "D?" V 4146 4082 50  0000 R CNN
+F 1 "D_Small" V 4055 4082 50  0000 R CNN
+F 2 "" V 4100 4150 50  0001 C CNN
+F 3 "~" V 4100 4150 50  0001 C CNN
+	1    4100 4150
+	0    -1   -1   0
+$EndComp
+Wire Wire Line
+	4100 4050 4200 4050
+$Comp
+L MX_Alps_Hybrid:MX-NoLED MX?
+U 1 1 65EEEAC1
+P 4750 3900
+F 0 "MX?" H 4783 4123 60  0000 C CNN
+F 1 "MX-NoLED" H 4783 4049 20  0000 C CNN
+F 2 "" H 4125 3875 60  0001 C CNN
+F 3 "" H 4125 3875 60  0001 C CNN
+	1    4750 3900
+	1    0    0    -1
+$EndComp
+$Comp
+L Device:D_Small D?
+U 1 1 65EEEAC7
+P 4600 4150
+F 0 "D?" V 4646 4082 50  0000 R CNN
+F 1 "D_Small" V 4555 4082 50  0000 R CNN
+F 2 "" V 4600 4150 50  0001 C CNN
+F 3 "~" V 4600 4150 50  0001 C CNN
+	1    4600 4150
+	0    -1   -1   0
+$EndComp
+Wire Wire Line
+	4600 4050 4700 4050
+$Comp
+L MX_Alps_Hybrid:MX-NoLED MX?
+U 1 1 65EEF2E3
+P 5250 3900
+F 0 "MX?" H 5283 4123 60  0000 C CNN
+F 1 "MX-NoLED" H 5283 4049 20  0000 C CNN
+F 2 "" H 4625 3875 60  0001 C CNN
+F 3 "" H 4625 3875 60  0001 C CNN
+	1    5250 3900
+	1    0    0    -1
+$EndComp
+$Comp
+L Device:D_Small D?
+U 1 1 65EEF2E9
+P 5100 4150
+F 0 "D?" V 5146 4082 50  0000 R CNN
+F 1 "D_Small" V 5055 4082 50  0000 R CNN
+F 2 "" V 5100 4150 50  0001 C CNN
+F 3 "~" V 5100 4150 50  0001 C CNN
+	1    5100 4150
+	0    -1   -1   0
+$EndComp
+Wire Wire Line
+	5100 4050 5200 4050
+$Comp
+L MX_Alps_Hybrid:MX-NoLED MX?
+U 1 1 65EF00BE
+P 4250 4550
+F 0 "MX?" H 4283 4773 60  0000 C CNN
+F 1 "MX-NoLED" H 4283 4699 20  0000 C CNN
+F 2 "" H 3625 4525 60  0001 C CNN
+F 3 "" H 3625 4525 60  0001 C CNN
+	1    4250 4550
+	1    0    0    -1
+$EndComp
+$Comp
+L Device:D_Small D?
+U 1 1 65EF00C4
+P 4100 4800
+F 0 "D?" V 4146 4732 50  0000 R CNN
+F 1 "D_Small" V 4055 4732 50  0000 R CNN
+F 2 "" V 4100 4800 50  0001 C CNN
+F 3 "~" V 4100 4800 50  0001 C CNN
+	1    4100 4800
+	0    -1   -1   0
+$EndComp
+Wire Wire Line
+	4100 4700 4200 4700
+$Comp
+L MX_Alps_Hybrid:MX-NoLED MX?
+U 1 1 65EF06F6
+P 4750 4550
+F 0 "MX?" H 4783 4773 60  0000 C CNN
+F 1 "MX-NoLED" H 4783 4699 20  0000 C CNN
+F 2 "" H 4125 4525 60  0001 C CNN
+F 3 "" H 4125 4525 60  0001 C CNN
+	1    4750 4550
+	1    0    0    -1
+$EndComp
+$Comp
+L Device:D_Small D?
+U 1 1 65EF06FC
+P 4600 4800
+F 0 "D?" V 4646 4732 50  0000 R CNN
+F 1 "D_Small" V 4555 4732 50  0000 R CNN
+F 2 "" V 4600 4800 50  0001 C CNN
+F 3 "~" V 4600 4800 50  0001 C CNN
+	1    4600 4800
+	0    -1   -1   0
+$EndComp
+Wire Wire Line
+	4600 4700 4700 4700
+$Comp
+L MX_Alps_Hybrid:MX-NoLED MX?
+U 1 1 65EF11E9
+P 5250 4550
+F 0 "MX?" H 5283 4773 60  0000 C CNN
+F 1 "MX-NoLED" H 5283 4699 20  0000 C CNN
+F 2 "" H 4625 4525 60  0001 C CNN
+F 3 "" H 4625 4525 60  0001 C CNN
+	1    5250 4550
+	1    0    0    -1
+$EndComp
+$Comp
+L Device:D_Small D?
+U 1 1 65EF11EF
+P 5100 4800
+F 0 "D?" V 5146 4732 50  0000 R CNN
+F 1 "D_Small" V 5055 4732 50  0000 R CNN
+F 2 "" V 5100 4800 50  0001 C CNN
+F 3 "~" V 5100 4800 50  0001 C CNN
+	1    5100 4800
+	0    -1   -1   0
+$EndComp
+Wire Wire Line
+	5100 4700 5200 4700
+$Comp
+L MX_Alps_Hybrid:The-Big-Switch U?
+U 1 1 65EF48DD
+P 3250 4050
+F 0 "U?" H 3308 4815 50  0000 C CNN
+F 1 "The-Big-Switch" H 3308 4724 50  0000 C CNN
+F 2 "" H 2700 4700 50  0001 C CNN
+F 3 "" H 2700 4700 50  0001 C CNN
+	1    3250 4050
+	1    0    0    -1
+$EndComp
+$Comp
+L MX_Alps_Hybrid:MX-NoLED MX?
+U 1 1 65F09C65
+P 4250 3250
+F 0 "MX?" H 4283 3473 60  0000 C CNN
+F 1 "MX-NoLED" H 4283 3399 20  0000 C CNN
+F 2 "" H 3625 3225 60  0001 C CNN
+F 3 "" H 3625 3225 60  0001 C CNN
+	1    4250 3250
+	1    0    0    -1
+$EndComp
+$Comp
+L Device:D_Small D?
+U 1 1 65F09C6B
+P 4100 3500
+F 0 "D?" V 4146 3432 50  0000 R CNN
+F 1 "D_Small" V 4055 3432 50  0000 R CNN
+F 2 "" V 4100 3500 50  0001 C CNN
+F 3 "~" V 4100 3500 50  0001 C CNN
+	1    4100 3500
+	0    -1   -1   0
+$EndComp
+Wire Wire Line
+	4100 3400 4200 3400
+$Comp
+L MX_Alps_Hybrid:MX-NoLED MX?
+U 1 1 65F09C72
+P 4750 3250
+F 0 "MX?" H 4783 3473 60  0000 C CNN
+F 1 "MX-NoLED" H 4783 3399 20  0000 C CNN
+F 2 "" H 4125 3225 60  0001 C CNN
+F 3 "" H 4125 3225 60  0001 C CNN
+	1    4750 3250
+	1    0    0    -1
+$EndComp
+$Comp
+L Device:D_Small D?
+U 1 1 65F09C78
+P 4600 3500
+F 0 "D?" V 4646 3432 50  0000 R CNN
+F 1 "D_Small" V 4555 3432 50  0000 R CNN
+F 2 "" V 4600 3500 50  0001 C CNN
+F 3 "~" V 4600 3500 50  0001 C CNN
+	1    4600 3500
+	0    -1   -1   0
+$EndComp
+Wire Wire Line
+	4600 3400 4700 3400
 $EndSCHEMATC
