File: hardware/micarrizo-pad.sch (KiCad schematic (older format))
At the start: 20 parts, among them U1 The-Big-Switch, U2 KB2040

Commit message: fix submodule
Parts:
- MX2, MX3, MX4, MX5, MX6, MX7, MX8: symbol MX_Alps_Hybrid:MX-NoLED -> micarrizo-pad-rescue:MX-NoLED-MX_Alps_Hybrid
- U1: symbol New_Library:The-Big-Switch -> The_Big_Switch:The-Big-Switch
- U2: symbol New_Library:KB2040 -> The_Big_Switch:KB2040
Changed lines of the file:
@@
 $EndDescr
 $Comp
-L MX_Alps_Hybrid:MX-NoLED MX3
+L micarrizo-pad-rescue:MX-NoLED-MX_Alps_Hybrid MX3
 U 1 1 65EE9E93
 P 5900 3500
@@
 	5750 3650 5850 3650
 $Comp
-L MX_Alps_Hybrid:MX-NoLED MX4
+L micarrizo-pad-rescue:MX-NoLED-MX_Alps_Hybrid MX4
 U 1 1 65EEEAC1
 P 6400 3500
@@
 	6250 3650 6350 3650
 $Comp
-L MX_Alps_Hybrid:MX-NoLED MX5
+L micarrizo-pad-rescue:MX-NoLED-MX_Alps_Hybrid MX5
 U 1 1 65EEF2E3
 P 6900 3500
@@
 	6750 3650 6850 3650
 $Comp
-L MX_Alps_Hybrid:MX-NoLED MX6
+L micarrizo-pad-rescue:MX-NoLED-MX_Alps_Hybrid MX6
 U 1 1 65EF00BE
 P 5900 4150
@@
 	6250 4300 6350 4300
 $Comp
-L MX_Alps_Hybrid:MX-NoLED MX8
+L micarrizo-pad-rescue:MX-NoLED-MX_Alps_Hybrid MX8
 U 1 1 65EF11E9
 P 6900 4150
@@
 	5750 3000 5850 3000
 $Comp
-L MX_Alps_Hybrid:MX-NoLED MX2
+L micarrizo-pad-rescue:MX-NoLED-MX_Alps_Hybrid MX2
 U 1 1 65F09C72
 P 6400 2850
@@
 	6250 3000 6350 3000
 $Comp
-L New_Library:The-Big-Switch U1
+L The_Big_Switch:The-Big-Switch U1
 U 1 1 65F2656C
 P 4800 3600
@@
 $EndComp
 $Comp
-L New_Library:KB2040 U2
+L The_Big_Switch:KB2040 U2
 U 1 1 65F497B3
 P 3250 3650
@@
 COL2
 $Comp
-L MX_Alps_Hybrid:MX-NoLED MX7
+L micarrizo-pad-rescue:MX-NoLED-MX_Alps_Hybrid MX7
 U 1 1 65EF06F6
 P 6400 4150

Commit message: finish reorganizing
Parts:
- MX2, MX4, MX5, MX6, MX7, MX8: symbol micarrizo-pad-rescue:MX-NoLED-MX_Alps_Hybrid -> micarrizo-pad-rescue:MX-NoLED-MX_Alps_Hybrid-micarrizo-pad-rescue
- MX3: symbol micarrizo-pad-rescue:MX-NoLED-MX_Alps_Hybrid -> MX_Alps_Hybrid:MX-NoLED
Changed lines of the file:
@@
 $EndDescr
 $Comp
-L micarrizo-pad-rescue:MX-NoLED-MX_Alps_Hybrid MX3
+L MX_Alps_Hybrid:MX-NoLED MX3
 U 1 1 65EE9E93
 P 5900 3500
@@
 	5750 3650 5850 3650
 $Comp
-L micarrizo-pad-rescue:MX-NoLED-MX_Alps_Hybrid MX4
+L micarrizo-pad-rescue:MX-NoLED-MX_Alps_Hybrid-micarrizo-pad-rescue MX4
 U 1 1 65EEEAC1
 P 6400 3500
@@
 	6250 3650 6350 3650
 $Comp
-L micarrizo-pad-rescue:MX-NoLED-MX_Alps_Hybrid MX5
+L micarrizo-pad-rescue:MX-NoLED-MX_Alps_Hybrid-micarrizo-pad-rescue MX5
 U 1 1 65EEF2E3
 P 6900 3500
@@
 	6750 3650 6850 3650
 $Comp
-L micarrizo-pad-rescue:MX-NoLED-MX_Alps_Hybrid MX6
+L micarrizo-pad-rescue:MX-NoLED-MX_Alps_Hybrid-micarrizo-pad-rescue MX6
 U 1 1 65EF00BE
 P 5900 4150
@@
 	6250 4300 6350 4300
 $Comp
-L micarrizo-pad-rescue:MX-NoLED-MX_Alps_Hybrid MX8
+L micarrizo-pad-rescue:MX-NoLED-MX_Alps_Hybrid-micarrizo-pad-rescue MX8
 U 1 1 65EF11E9
 P 6900 4150
@@
 	5750 3000 5850 3000
 $Comp
-L micarrizo-pad-rescue:MX-NoLED-MX_Alps_Hybrid MX2
+L micarrizo-pad-rescue:MX-NoLED-MX_Alps_Hybrid-micarrizo-pad-rescue MX2
 U 1 1 65F09C72
 P 6400 2850
@@
 COL2
 $Comp
-L micarrizo-pad-rescue:MX-NoLED-MX_Alps_Hybrid MX7
+L micarrizo-pad-rescue:MX-NoLED-MX_Alps_Hybrid-micarrizo-pad-rescue MX7
 U 1 1 65EF06F6
 P 6400 4150
